File: attiny1616_linetracker.kicad_pcb (KiCad board)
At the start: 2 copper layers, 72.6 x 48.8 mm, 16 parts, among them J1 Auriga_JST, J2 ATtiny_L, J3 ATtiny_R, J4 IR_TRACKER, J5 Conn_01x08_Socket, J6 Conn_01x04_Socket, J7 Conn_01x04_Socket, M7 MountingHole_3.2mm_M3, M8 MountingHole_3.2mm_M3

Commit message: Preproduction
Parts:
- D1: footprint Diode_SMD:D_1206_3216Metric -> PCM_Diode_SMD_AKL:D_SOD-123
Connections:
- net Net-(D1-A) renamed /V_{in}
