File: attiny1616_linetracker.kicad_sch (KiCad schematic)
At the start: 14 parts, among them J1 Auriga_JST, J2 ATtiny_L, J3 ATtiny_R, J4 IR_TRACKER, J5 Conn_01x08_Socket, J6 Conn_01x04_Socket, J7 Conn_01x04_Socket

Commit message: Preproduction
Parts:
- D1: footprint Diode_SMD:D_1206_3216Metric -> PCM_Diode_SMD_AKL:D_SOD-123; symbol Device:D_Schottky -> PCM_Diode_Schottky_AKL:BAT65; LCSC (none) -> C78545
- J1: LCSC (none) -> C157919
- J2, J3: LCSC (none) -> C2897373
- J4: LCSC (none) -> C6332200
- J5: LCSC (none) -> C27438
- J6, J7: LCSC (none) -> C2718488
Connections:
- net V_{in}: now reaches D1.2 (A), J1.4 (PWR_B)
Changed lines of the file:
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@@
 		)
 	)
-	(label "IR2"
-		(at 100.33 78.74 0)
+	(label "GND"
+		(at 179.07 74.93 0)
 		(fields_autoplaced yes)
 		(effects
@@
 		)
 	)
-	(label "SDA"
-		(at 179.07 72.39 0)
+	(label "IR2"
+		(at 100.33 78.74 0)
 		(fields_autoplaced yes)
 		(effects
@@
 		)
 	)
-	(label "GND"
-		(at 100.33 73.66 0)
+	(label "SDA"
+		(at 179.07 72.39 0)
 		(fields_autoplaced yes)
 		(effects
@@
 		)
 	)
-	(label "V_{cc}"
-		(at 100.33 71.12 0)
+	(label "GND"
+		(at 100.33 73.66 0)
 		(fields_autoplaced yes)
 		(effects
@@
 		)
 	)
-	(label "S2"
-		(at 179.07 82.55 0)
+	(label "V_{in}"
+		(at 179.07 77.47 0)
 		(fields_autoplaced yes)
 		(effects
@@
 		)
 	)
-	(label "IR5"
-		(at 100.33 86.36 0)
+	(label "V_{cc}"
+		(at 100.33 71.12 0)
 		(fields_autoplaced yes)
 		(effects
@@
 		)
 	)
-	(label "IR1"
-		(at 100.33 76.2 0)
+	(label "S2"
+		(at 179.07 82.55 0)
 		(fields_autoplaced yes)
 		(effects
@@
 		)
 	)
-	(label "IR4"
-		(at 100.33 83.82 0)
+	(label "IR5"
+		(at 100.33 86.36 0)
 		(fields_autoplaced yes)
 		(effects
@@
 		)
 	)
-	(label "SCL"
-		(at 179.07 69.85 0)
+	(label "IR1"
+		(at 100.33 76.2 0)
 		(fields_autoplaced yes)
 		(effects
@@
 		)
 	)
+	(label "IR4"
+		(at 100.33 83.82 0)
+		(fields_autoplaced yes)
+		(effects
+			(font
+				(size 1.27 1.27)
+			)
+			(justify left bottom)
+		)
+	)
+	(label "SCL"
+		(at 179.07 69.85 0)
+		(fields_autoplaced yes)
+		(effects
+			(font
+				(size 1.27 1.27)
+			)
+			(justify left bottom)
+		)
+	)
 	(symbol
 		(lib_id "Connector_Generic:Conn_01x10")
@@
 			)
 		)
+		(property "LCSC" "C2897373"
+			(at 154.94 80.01 0)
+			(effects
+				(font
+					(size 1.27 1.27)
+				)
+				(hide yes)
+			)
+		)
 		(pin "1"
 		)
@@
 			)
 		)
+		(property "LCSC" "C27438"
+			(at 142.24 129.54 90)
+			(effects
+				(font
+					(size 1.27 1.27)
+				)
+				(hide yes)
+			)
+		)
 		(pin "8"
 		)
@@
 		)
 		(property "Description" "Generic connector, single row, 01x04, script generated"
+			(at 190.5 27.94 0)
+			(effects
+				(font
+					(size 1.27 1.27)
+				)
+				(hide yes)
+			)
+		)
+		(property "LCSC" "C2718488"
 			(at 190.5 27.94 0)
 			(effects
@@
 			)
 		)
+		(property "LCSC" "C6332200"
+			(at 93.98 78.74 0)
+			(effects
+				(font
+					(size 1.27 1.27)
+				)
+				(hide yes)
+			)
+		)
 		(pin "6"
 		)
@@
 			)
 		)
+		(property "LCSC" "C2718488"
+			(at 190.5 41.91 0)
+			(effects
+				(font
+					(size 1.27 1.27)
+				)
+				(hide yes)
+			)
+		)
 		(pin "4"
 		)
@@
 		(property "Description" "Generic connector, single row, 01x06, script generated (kicad-library-utils/schlib/autogen/connector/)"
 			(at 188.214 85.598 0)
+			(effects
+				(font
+					(size 1.27 1.27)
+				)
+				(hide yes)
+			)
+		)
+		(property "LCSC" "C157919"
+			(at 187.96 74.93 0)
 			(effects
 				(font
@@
 			)
 		)
+		(property "LCSC" "C2897373"
+			(at 125.73 80.01 0)
+			(effects
+				(font
+					(size 1.27 1.27)
+				)
+				(hide yes)
+			)
+		)
 		(pin "1"
 		)
@@
 	)
 	(symbol
-		(lib_id "Device:D_Schottky")
-		(at 167.64 64.77 0)
+		(lib_id "PCM_Diode_Schottky_AKL:BAT65")
+		(at 167.64 64.77 180)
 		(unit 1)
 		(exclude_from_sim no)
@@
 			)
 		)
-		(property "Footprint" "Diode_SMD:D_1206_3216Metric"
+		(property "Footprint" "PCM_Diode_SMD_AKL:D_SOD-123"
 			(at 167.64 64.77 0)
 			(effects
@@
 			)
 		)
-		(property "Datasheet" "~"
+		(property "Datasheet" "https://pdf.datasheetcatalog.com/datasheet/siemens/BAT65.pdf"
 			(at 167.64 64.77 0)
 			(effects
@@
 			)
 		)
-		(property "Description" "Schottky diode"
+		(property "Description" "SOD-123 Schottky diode, 40V, 500mA, Alternate KiCAD Library"
 			(at 167.64 64.77 0)
 			(effects
+				(font
+					(size 1.27 1.27)
+				)
+				(hide yes)
+			)
+		)
+		(property "LCSC" "C78545"
+			(at 167.64 64.77 0)
+			(effects
